Commit message: updated cart length

File: data/robot_description/abb_linear_axis/urdf/abb_robot_plattform.urdf (robot description, URDF)
Before this commit: robot abb_irb6700_linear_axis, 15 links, 14 joints
Joints:
- joint axis_joint: limit lower=0.0 upper=5.0 effort=100000 velocity=2.618 -> lower=0.0 upper=4.2 effort=100000 velocity=2.618
